File: Hardware/board_final/hydrophone_stm32_board.sch (KiCad schematic (older format))
At the start: 101 parts, among them IC1 AD8031ARZ, J1 Conn_01x02, J2 Conn_02x05_Odd_Even, J3 Conn_01x02, J4 Conn_01x03, J5 47352-1001, J6 142-0701-851, J7 Conn_01x02_Female, U1 AMS1117-3.3, U2 STM32F746ZGT6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

Commit message: Added F7 100 Pin Version
Parts:
- removed C1: 4.7u, Capacitor_Tantalum_SMD:CP_EIA-3216-18_Kemet-A, symbol Device:CP1_Small
- removed C28, C29: 18p, Capacitor_SMD:C_0402_1005Metric, symbol Device:C_Small
- removed C3: 1u, Capacitor_Tantalum_SMD:CP_EIA-3216-18_Kemet-A, symbol Device:CP1_Small
- removed HSE1: 25MHz, Crystal:Crystal_SMD_3225-4Pin_3.2x2.5mm, symbol Device:Crystal_GND24_Small
- removed J5: 47352-1001, 47352-1001, symbol SamacSys_Parts:47352-1001
- removed R10: 47k, Resistor_SMD:R_0402_1005Metric, symbol Device:R_Small_US
- removed R2: 100, Resistor_SMD:R_0402_1005Metric, symbol Device:R_Small
- added C1, C3: 4.3p, Capacitor_SMD:C_0402_1005Metric, symbol Device:C_Small
- added J5: Micro_SD_Card, Connector_Card:microSD_HC_Hirose_DM3AT-SF-PEJM5, symbol Connector:Micro_SD_Card
- added R2: 47k, Resistor_SMD:R_0402_1005Metric, symbol Device:R_Small_US
- added Y1: Crystal, SamacSys_Parts:RESC3226X100N, symbol Device:Crystal
- J4: value Conn_01x03 -> Conn_01x04; footprint Connector_PinHeader_2.54mm:PinHeader_1x03_P2.54mm_Vertical -> Connector_PinHeader_2.54mm:PinHeader_1x04_P2.54mm_Vertical; symbol Connector_Generic:Conn_01x03 -> Connector_Generic:Conn_01x04
Connections:
- net +3V3: now also J4.3 (Pin_3), R5.2, J5.4 (VDD), R2.2; no longer IC1.7 (+VS), R5.1
- net GND: now also J4.4 (Pin_4), C1.2, C3.2, J5.6 (VSS), J5.9 (SHIELD); no longer J4.3 (Pin_3)
- net PDR_ON: now also R5.1; no longer R5.2
- net uSD_CLK: now also J5.5 (CLK)
- net uSD_CMD: now also J5.3 (CMD)
- net uSD_D0: now also J5.7 (DAT0), R2.1
- net uSD_D1: now also J5.8 (DAT1)
- net uSD_D2: now also J5.1 (DAT2)
- net uSD_D3: now also J5.2 (DAT3/CD)
- net HSE_IN: no longer names the net of U2.23 (PH0)
- net HSE_IN: now also C1.1, Y1.1
- net HSE_OUT: no longer names the net of U2.24 (PH1)
- net HSE_OUT: now also C3.1, Y1.2
- net VREF renamed VDIV
Other:
- moved on the sheet: C2, R3, R4, R5, R6, R7, R8
