File: CM4IO/CM4/CM4.kicad_pcb (KiCad board)
At the start: 4 copper layers, 113 parts, among them IC1 OPA659IDBVR, IC2 OPA659IDBVR, IC3 LMH6643MAX_NOPB, IC4 TPS65133DPDR, IC5 TPS62111RSAT, IC6 STM32H747IIT6, J1 901-144-8RFX, J2 USB_C_Receptacle_USB2.0, J3 SWDIO, J4 Micro_SD_Card, J5 DJI UART, Q1 AO3401A, SW1 SW_SPDT, U1 USBLC6-2SC6, Y1 16MHz, Y2 32.768KHz

Commit message: Completed H7/CM4IO Board
Parts:
- removed L5: 39n, Inductor_SMD:L_0402_1005Metric
- removed SW1: SW_SPDT, Button_Switch_SMD:SW_SPDT_PCM12
- removed U1: USBLC6-2SC6, Package_TO_SOT_SMD:SOT-23-6
- added FB2: 100 @ 100 MHz, Inductor_SMD:L_0603_1608Metric, F.Cu at (97.8, 119.1)
- added J6: Conn_01x02_Female, Connector_PinHeader_2.54mm:PinHeader_1x02_P2.54mm_Horizontal, F.Cu at (79.3, 93.1)
- C1, C2, C3, C4, C5, IC1, IC2, IC3, J5, Module1, R1, R10, R11, R12, R13, R14, R15, R16, R2, R3, R4, R5, R6, R7, R8, R9: moved to B.Cu
- J1: value 901-144-8RFX -> Conn_Coaxial; footprint SamacSys_Parts:9011448RFX -> Connector_Coaxial:SMA_Samtec_SMA-J-P-H-ST-EM1_EdgeMount; moved to B.Cu
- R18: value 0 -> 47
- moved J5 41.4 mm to (115.4, 84.3), turned to 0 degrees
- moved J3 31.0 mm to (127.8, 83.9), turned to -90 degrees
- moved Module1 28.6 mm to (135.7, 90.4), turned to -90 degrees
- moved R5 17.3 mm to (95.9, 95.4)
- moved R16 15.7 mm to (136.8, 133.3), turned to -90 degrees
- moved C4 15.3 mm to (93.9, 91.2)
- moved R4 15.0 mm to (93.1, 88.3)
- moved R10 14.4 mm to (92.9, 98.7), turned to 180 degrees
- moved R2 13.5 mm to (94.5, 93.2), turned to 90 degrees
- moved S1 13.5 mm to (146.4, 119.6)
- moved J1 13.4 mm to (92.6, 84.7), turned to 90 degrees
- moved C2 13.2 mm to (93.9, 89.7), turned to 0 degrees
- moved H1 12.3 mm to (78.6, 132.0)
- moved FB1 12.1 mm to (125.9, 124.7), turned to 90 degrees
- moved H2 12.1 mm to (78.4, 85.5)
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Connections:
- C48 pad 2: /H7MCU/HSE_IN -> Net-(C48-Pad2)
- C49 pad 1: Net-(C49-Pad1) -> /H7MCU/HSE_IN
- J2 pad A6: /Power/USB_CONN_D+ -> Net-(J2-PadA6)
- J2 pad A7: /Power/USB_CONN_D- -> Net-(J2-PadA7)
- J2 pad B6: /Power/USB_CONN_D+ -> Net-(J2-PadB6)
- J2 pad B7: /Power/USB_CONN_D- -> Net-(J2-PadB7)
- R20 pad 2: Net-(C49-Pad1) -> Net-(C48-Pad2)
- R27 pad 2: Net-(R27-Pad2) -> GND
- Y1 pad 1: Net-(C49-Pad1) -> /H7MCU/HSE_IN
- Y1 pad 3: /H7MCU/HSE_IN -> Net-(C48-Pad2)
Routing:
- net GND: track 0.00 -> 402.2 mm, vias 0 -> 133
- net /+3.3V: track 0.00 -> 174.7 mm, vias 0 -> 58
- net /5V: track 0.00 -> 163.3 mm, vias 0 -> 10
- net /H7MCU/NRST: track 0.00 -> 115.7 mm, vias 0 -> 4
- net /VPOS: track 0.00 -> 99.8 mm, vias 0 -> 1
- net /VNEG: track 0.00 -> 83.9 mm, vias 0 -> 4
- net Net-(BT1-Pad1): track 0.00 -> 63.4 mm, vias 0 -> 2
- net /v_DIV_OUT: track 0.00 -> 58.1 mm, vias 0 -> 4
- net /USB_D+: track 0.00 -> 44.8 mm, vias 0 -> 1
- net /STM32_3_RX: track 0.00 -> 43.4 mm, vias 0 -> 1
- net /USB_D-: track 0.00 -> 42.8 mm, vias 0 -> 1
- net /STM32_3_TX: track 0.00 -> 29.4 mm, vias 0 -> 3
- net /H7MCU/SDMMC_D1: track 0.00 -> 26.7 mm, vias 0 -> 2
- net VCC: track 0.00 -> 26.6 mm
- net /H7MCU/SDMMC_CK: track 0.00 -> 25.6 mm, vias 0 -> 2
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- added copper zone on In2.Cu, net /+3.3V
- added copper zone on In1.Cu, net GND
Other:
- board outline added: 76.2 x 54.3 mm
