File: CM4IO/CM4/_autosave-CM4.kicad_pcb (KiCad board)
At the start: 4 copper layers, 76.2 x 54.3 mm, 113 parts, among them IC1 OPA659IDBVR, IC2 OPA659IDBVR, IC3 LMH6643MAX_NOPB, IC4 TPS65133DPDR, IC5 TPS62111RSAT, IC6 STM32H747IIT6, J1 Conn_Coaxial, J2 USB_C_Receptacle_USB2.0, J3 SWDIO, J4 Micro_SD_Card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

Commit message: Corrected SMPS configuration
Changed lines of the file:
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@@
       (plotinvisibletext false)
       (sketchpadsonfab false)
-      (subtractmaskfromsilk false)
+      (subtractmaskfromsilk true)
       (outputformat 1)
       (mirror false)
-      (drillshape 1)
+      (drillshape 0)
       (scaleselection 1)
-      (outputdirectory "")
+      (outputdirectory "gerber/")
     )
   )
@@
     (fp_line (start 1.6 0.8) (end 1.6 -0.8) (layer "F.Fab") (width 0.1))
     (fp_line (start 1.6 -0.8) (end -1.2 -0.8) (layer "F.Fab") (width 0.1))
-    (pad "1" smd roundrect (at -1.35 0 270) (size 1.4 1.35) (layers "F.Cu" "F.Paste" "F.Mask") (roundrect_rratio 0.185185)
+    (pad "1" smd roundrect (at -1.35 0 270) (size 1.4 1.35) (layers "F.Cu" "F.Paste" "F.Mask") (roundrect_rratio 0.1851851851851852)
       (net 14 "/H7MCU/+3.3VA"))
-    (pad "2" smd roundrect (at 1.35 0 270) (size 1.4 1.35) (layers "F.Cu" "F.Paste" "F.Mask") (roundrect_rratio 0.185185)
+    (pad "2" smd roundrect (at 1.35 0 270) (size 1.4 1.35) (layers "F.Cu" "F.Paste" "F.Mask") (roundrect_rratio 0.1851851851851852)
       (net 1 "GND"))
     (model "${KISYS3DMOD}/Capacitor_Tantalum_SMD.3dshapes/CP_EIA-3216-18_Kemet-A.wrl"
@@
     (fp_line (start 1.6 -1.25) (end 1.6 1.25) (layer "F.Fab") (width 0.1))
     (fp_line (start 1.6 1.25) (end -1.6 1.25) (layer "F.Fab") (width 0.1))
-    (pad "1" smd roundrect (at -1.475 0 270) (size 1.15 2.7) (layers "F.Cu" "F.Paste" "F.Mask") (roundrect_rratio 0.217391)
+    (pad "1" smd roundrect (at -1.475 0 270) (size 1.15 2.7) (layers "F.Cu" "F.Paste" "F.Mask") (roundrect_rratio 0.2173913043478261)
       (net 12 "/+3.3V"))
-    (pad "2" smd roundrect (at 1.475 0 270) (size 1.15 2.7) (layers "F.Cu" "F.Paste" "F.Mask") (roundrect_rratio 0.217391)
+    (pad "2" smd roundrect (at 1.475 0 270) (size 1.15 2.7) (layers "F.Cu" "F.Paste" "F.Mask") (roundrect_rratio 0.2173913043478261)
       (net 1 "GND"))
     (model "${KISYS3DMOD}/Capacitor_SMD.3dshapes/C_1210_3225Metric.wrl"
@@
     (fp_line (start -1 -0.625) (end 1 -0.625) (layer "F.Fab") (width 0.1))
     (fp_line (start -1 0.625) (end -1 -0.625) (layer "F.Fab") (width 0.1))
-    (pad "1" smd roundrect (at -0.9125 0) (size 1.025 1.4) (layers "F.Cu" "F.Paste" "F.Mask") (roundrect_rratio 0.243902)
+    (pad "1" smd roundrect (at -0.9125 0) (size 1.025 1.4) (layers "F.Cu" "F.Paste" "F.Mask") (roundrect_rratio 0.2439024390243902)
       (net 40 "/Power/PG"))
-    (pad "2" smd roundrect (at 0.9125 0) (size 1.025 1.4) (layers "F.Cu" "F.Paste" "F.Mask") (roundrect_rratio 0.243902)
+    (pad "2" smd roundrect (at 0.9125 0) (size 1.025 1.4) (layers "F.Cu" "F.Paste" "F.Mask") (roundrect_rratio 0.2439024390243902)
       (net 12 "/+3.3V"))
     (model "${KISYS3DMOD}/Resistor_SMD.3dshapes/R_0805_2012Metric.wrl"
@@
     (fp_line (start -1.2 -0.8) (end -1.6 -0.4) (layer "F.Fab") (width 0.1))
     (fp_line (start 1.6 0.8) (end 1.6 -0.8) (layer "F.Fab") (width 0.1))
-    (pad "1" smd roundrect (at -1.35 0 90) (size 1.4 1.35) (layers "F.Cu" "F.Paste" "F.Mask") (roundrect_rratio 0.185185)
+    (pad "1" smd roundrect (at -1.35 0 90) (size 1.4 1.35) (layers "F.Cu" "F.Paste" "F.Mask") (roundrect_rratio 0.1851851851851852)
       (net 12 "/+3.3V"))
-    (pad "2" smd roundrect (at 1.35 0 90) (size 1.4 1.35) (layers "F.Cu" "F.Paste" "F.Mask") (roundrect_rratio 0.185185)
+    (pad "2" smd roundrect (at 1.35 0 90) (size 1.4 1.35) (layers "F.Cu" "F.Paste" "F.Mask") (roundrect_rratio 0.1851851851851852)
       (net 1 "GND"))
     (model "${KISYS3DMOD}/Capacitor_Tantalum_SMD.3dshapes/CP_EIA-3216-18_Kemet-A.wrl"
@@
     (fp_line (start -1.6 1.25) (end -1.6 -1.25) (layer "F.Fab") (width 0.1))
     (fp_line (start 1.6 -1.25) (end 1.6 1.25) (layer "F.Fab") (width 0.1))
-    (pad "1" smd roundrect (at -1.475 0 270) (size 1.15 2.7) (layers "F.Cu" "F.Paste" "F.Mask") (roundrect_rratio 0.217391)
+    (pad "1" smd roundrect (at -1.475 0 270) (size 1.15 2.7) (layers "F.Cu" "F.Paste" "F.Mask") (roundrect_rratio 0.2173913043478261)
       (net 9 "/5V"))
-    (pad "2" smd roundrect (at 1.475 0 270) (size 1.15 2.7) (layers "F.Cu" "F.Paste" "F.Mask") (roundrect_rratio 0.217391)
+    (pad "2" smd roundrect (at 1.475 0 270) (size 1.15 2.7) (layers "F.Cu" "F.Paste" "F.Mask") (roundrect_rratio 0.2173913043478261)
       (net 1 "GND"))
     (model "${KISYS3DMOD}/Capacitor_SMD.3dshapes/C_1210_3225Metric.wrl"
@@
     (fp_line (start -1.6 -0.4) (end -1.6 0.8) (layer "F.Fab") (width 0.1))
     (fp_line (start -1.2 -0.8) (end -1.6 -0.4) (layer "F.Fab") (width 0.1))
-    (pad "1" smd roundrect (at -1.35 0) (size 1.4 1.35) (layers "F.Cu" "F.Paste" "F.Mask") (roundrect_rratio 0.185185)
+    (pad "1" smd roundrect (at -1.35 0) (size 1.4 1.35) (layers "F.Cu" "F.Paste" "F.Mask") (roundrect_rratio 0.1851851851851852)
       (net 15 "/H7MCU/VCAP1"))
-    (pad "2" smd roundrect (at 1.35 0) (size 1.4 1.35) (layers "F.Cu" "F.Paste" "F.Mask") (roundrect_rratio 0.185185)
+    (pad "2" smd roundrect (at 1.35 0) (size 1.4 1.35) (layers "F.Cu" "F.Paste" "F.Mask") (roundrect_rratio 0.1851851851851852)
       (net 1 "GND"))
     (model "${KISYS3DMOD}/Capacitor_Tantalum_SMD.3dshapes/CP_EIA-3216-18_Kemet-A.wrl"
@@
     (fp_line (start 1.6 0.8) (end 1.6 -0.8) (layer "F.Fab") (width 0.1))
     (fp_line (start 1.6 -0.8) (end -1.2 -0.8) (layer "F.Fab") (width 0.1))
-    (pad "1" smd roundrect (at -1.35 0 180) (size 1.4 1.35) (layers "F.Cu" "F.Paste" "F.Mask") (roundrect_rratio 0.185185)
+    (pad "1" smd roundrect (at -1.35 0 180) (size 1.4 1.35) (layers "F.Cu" "F.Paste" "F.Mask") (roundrect_rratio 0.1851851851851852)
       (net 13 "/H7MCU/VREF+"))
-    (pad "2" smd roundrect (at 1.35 0 180) (size 1.4 1.35) (layers "F.Cu" "F.Paste" "F.Mask") (roundrect_rratio 0.185185)
+    (pad "2" smd roundrect (at 1.35 0 180) (size 1.4 1.35) (layers "F.Cu" "F.Paste" "F.Mask") (roundrect_rratio 0.1851851851851852)
       (net 1 "GND"))
     (model "${KISYS3DMOD}/Capacitor_Tantalum_SMD.3dshapes/CP_EIA-3216-18_Kemet-A.wrl"
@@
     (fp_line (start -1.6 -0.8) (end -1.6 0.8) (layer "B.Fab") (width 0.1))
     (fp_line (start 1.6 0.8) (end 1.6 -0.8) (layer "B.Fab") (width 0.1))
-    (pad "1" smd roundrect (at -1.4625 0 270) (size 1.125 1.75) (layers "B.Cu" "B.Paste" "B.Mask") (roundrect_rratio 0.222222)
+    (pad "1" smd roundrect (at -1.4625 0 270) (size 1.125 1.75) (layers "B.Cu" "B.Paste" "B.Mask") (roundrect_rratio 0.2222222222222222)
       (net 159 "Net-(J2-PadA5)"))
-    (pad "2" smd roundrect (at 1.4625 0 270) (size 1.125 1.75) (layers "B.Cu" "B.Paste" "B.Mask") (roundrect_rratio 0.222222)
+    (pad "2" smd roundrect (at 1.4625 0 270) (size 1.125 1.75) (layers "B.Cu" "B.Paste" "B.Mask") (roundrect_rratio 0.2222222222222222)
       (net 1 "GND"))
     (model "${KISYS3DMOD}/Resistor_SMD.3dshapes/R_1206_3216Metric.wrl"
@@
     (pad "3" smd roundrect (at 1.25 2.4) (size 0.8 1.6) (layers "B.Cu" "B.Paste" "B.Mask") (roundrect_rratio 0.25)
       (net 1 "GND") (pinfunction "Pin_3"))
-    (pad "MP" smd roundrect (at 3.8 -0.5) (size 2.1 3) (layers "B.Cu" "B.Paste" "B.Mask") (roundrect_rratio 0.119048))
-    (pad "MP" smd roundrect (at -3.8 -0.5) (size 2.1 3) (layers "B.Cu" "B.Paste" "B.Mask") (roundrect_rratio 0.119048))
+    (pad "MP" smd roundrect (at 3.8 -0.5) (size 2.1 3) (layers "B.Cu" "B.Paste" "B.Mask") (roundrect_rratio 0.1190480952380952))
+    (pad "MP" smd roundrect (at -3.8 -0.5) (size 2.1 3) (layers "B.Cu" "B.Paste" "B.Mask") (roundrect_rratio 0.1190480952380952))
     (model "${KISYS3DMOD}/Connector_Molex.3dshapes/Molex_PicoBlade_53261-0371_1x03-1MP_P1.25mm_Horizontal.wrl"
       (offset (xyz 0 0 0))
@@
     (fp_line (start 1.6 0.8) (end 1.6 -0.8) (layer "B.Fab") (width 0.1))
     (fp_line (start -1.6 0.8) (end 1.6 0.8) (layer "B.Fab") (width 0.1))
-    (pad "1" smd roundrect (at -1.4625 0 270) (size 1.125 1.75) (layers "B.Cu" "B.Paste" "B.Mask") (roundrect_rratio 0.222222)
+    (pad "1" smd roundrect (at -1.4625 0 270) (size 1.125 1.75) (layers "B.Cu" "B.Paste" "B.Mask") (roundrect_rratio 0.2222222222222222)
       (net 157 "Net-(J2-PadB5)"))
-    (pad "2" smd roundrect (at 1.4625 0 270) (size 1.125 1.75) (layers "B.Cu" "B.Paste" "B.Mask") (roundrect_rratio 0.222222)
+    (pad "2" smd roundrect (at 1.4625 0 270) (size 1.125 1.75) (layers "B.Cu" "B.Paste" "B.Mask") (roundrect_rratio 0.2222222222222222)
       (net 1 "GND"))
     (model "${KISYS3DMOD}/Resistor_SMD.3dshapes/R_1206_3216Metric.wrl"
